File: Arduino HackBo/hackbo.sch (KiCad schematic (older format))
At the start: 10 parts, among them IC1 ATMEGA168-A, P1 CONN_8, P2 CONN_6, P3 CONN_8, X1 CRYSTAL

Commit message: Adicionado Reset y Alimentación (HackBo 2014-08-26)
- Se adicionó el circuito de reset y las conexiones para la
alimentación.
- Se eliminaron componentes no utilizados.
- Se generaron los archivos GERBER.
Parts:
- added C6: 0.1uF, SM0603, symbol C
- added R1: 10k, SM0603, symbol R
- added SW1: SW_PUSH, SW_PUSH_SMALL, symbol SW_PUSH
Connections:
- net labels added: DTR, Reset
- wire segments 58 -> 69
Changed lines of the file:
@@
 Sheet 1 1
 Title ""
-Date "14 aug 2014"
+Date "27 aug 2014"
 Rev ""
 Comp ""
@@
 Text Label 5700 3000 0    60   ~ 0
 A1
+$Comp
+L SW_PUSH SW1
+U 1 1 53FD203A
+P 6750 1900
+F 0 "SW1" H 6900 2010 50  0000 C CNN
+F 1 "SW_PUSH" H 6750 1820 50  0000 C CNN
+F 2 "SW_PUSH_SMALL" H 6750 1900 60  0001 C CNN
+F 3 "~" H 6750 1900 60  0000 C CNN
+	1    6750 1900
+	0    -1   -1   0
+$EndComp
+$Comp
+L C C6
+U 1 1 53FD2047
+P 5850 1500
+F 0 "C6" H 5850 1600 40  0000 L CNN
+F 1 "0.1uF" H 5856 1415 40  0000 L CNN
+F 2 "SM0603" H 5888 1350 30  0000 C CNN
+F 3 "~" H 5850 1500 60  0000 C CNN
+	1    5850 1500
+	0    -1   -1   0
+$EndComp
+$Comp
+L GND #PWR09
+U 1 1 53FD204D
+P 6750 2400
+F 0 "#PWR09" H 6750 2400 30  0001 C CNN
+F 1 "GND" H 6750 2330 30  0001 C CNN
+F 2 "" H 6750 2400 60  0000 C CNN
+F 3 "" H 6750 2400 60  0000 C CNN
+	1    6750 2400
+	1    0    0    -1
+$EndComp
+$Comp
+L VCC #PWR010
+U 1 1 53FD2053
+P 6750 750
+F 0 "#PWR010" H 6750 850 30  0001 C CNN
+F 1 "VCC" H 6750 850 30  0000 C CNN
+F 2 "" H 6750 750 60  0000 C CNN
+F 3 "" H 6750 750 60  0000 C CNN
+	1    6750 750
+	1    0    0    -1
+$EndComp
+$Comp
+L R R1
+U 1 1 53FD205B
+P 6750 1100
+F 0 "R1" V 6830 1100 40  0000 C CNN
+F 1 "10k" V 6757 1101 40  0000 C CNN
+F 2 "SM0603" V 6680 1100 30  0001 C CNN
+F 3 "~" H 6750 1100 30  0000 C CNN
+	1    6750 1100
+	1    0    0    -1
+$EndComp
+Wire Wire Line
+	3500 2850 3750 2850
+Text Label 3550 2850 0    60   ~ 0
+Reset
+Wire Wire Line
+	6050 1500 7100 1500
+Connection ~ 6750 1500
+Connection ~ 6150 1500
+Wire Wire Line
+	6750 2400 6750 2200
+Wire Wire Line
+	6750 850  6750 750
+Wire Wire Line
+	6750 1350 6750 1600
+Text Label 6800 1500 0    60   ~ 0
+Reset
+Wire Wire Line
+	5650 1500 5350 1500
+Text Label 5400 1500 0    60   ~ 0
+DTR
+Wire Wire Line
+	4850 4400 4600 4400
+Text Label 4650 4400 0    60   ~ 0
+DTR
+$Comp
+L VCC #PWR011
+U 1 1 53FD2C41
+P 5750 3300
+F 0 "#PWR011" H 5750 3400 30  0001 C CNN
+F 1 "VCC" H 5750 3400 30  0000 C CNN
+F 2 "" H 5750 3300 60  0000 C CNN
+F 3 "" H 5750 3300 60  0000 C CNN
+	1    5750 3300
+	0    -1   -1   0
+$EndComp
+$Comp
+L GND #PWR012
+U 1 1 53FD2C93
+P 5700 3100
+F 0 "#PWR012" H 5700 3100 30  0001 C CNN
+F 1 "GND" H 5700 3030 30  0001 C CNN
+F 2 "" H 5700 3100 60  0000 C CNN
+F 3 "" H 5700 3100 60  0000 C CNN
+	1    5700 3100
+	0    1    1    0
+$EndComp
+Wire Wire Line
+	5900 3100 5700 3100
+Wire Wire Line
+	5750 3300 5900 3300
+Wire Wire Line
+	5900 3200 5850 3200
+Wire Wire Line
+	5850 3200 5850 3100
+Connection ~ 5850 3100
 $EndSCHEMATC
